File: Hardware/matrix_badge/matrix_badge.sch (KiCad schematic (older format))
At the start: 32 parts, among them J1 Conn_02x03_Odd_Even, U1 ATTINY85-20SU

Commit message: Made fixes for v02 (added wide body SOIC and swapped round pin for rectangular pin back). Added ON/OFF silk for v03.
Parts:
- U1: footprint digikey-footprints:SOIC-8_W5.3mm -> Package_SO:SOIJ-8_5.3x5.3mm_P1.27mm
Changed lines of the file:
@@
 EESchema Schematic File Version 4
+LIBS:matrix_badge-cache
 EELAYER 26 0
 EELAYER END
@@
 F 0 "U1" H 3578 3603 60  0000 L CNN
 F 1 "ATTINY85-20SU" H 3578 3497 60  0000 L CNN
-F 2 "digikey-footprints:SOIC-8_W5.3mm" H 3550 3900 60  0001 L CNN
+F 2 "Package_SO:SOIJ-8_5.3x5.3mm_P1.27mm" H 3550 3900 60  0001 L CNN
 F 3 "http://www.microchip.com/mymicrochip/filehandler.aspx?ddocname=en589894" H 3550 4000 60  0001 L CNN
 F 4 "ATTINY85-20SU-ND" H 3550 4100 60  0001 L CNN "Digi-Key_PN"
